File: brd/master/power-supply.sch (KiCad schematic (older format))
At the start: 35 parts, among them K1 5v DPDT, P1 IEC C13, Q1 BC547, T1 15-0-15 30VA, U5 LM7805CT, U6 LM7805CT, U7 LM7812CT, U8 LM7815CT, U9 LM7915CT

Commit message: slave version rc3
Connections:
- net at C19.1, C21.1, C23.1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: now also R44.1
Changed lines of the file:
@@
 LIBS:valves
 LIBS:master-cache
-EELAYER 24 0
+EELAYER 25 0
 EELAYER END
 $Descr A4 11693 8268
@@
 Wire Wire Line
 	8350 4350 9650 4350
+Wire Wire Line
+	6400 4250 6400 4200
 $EndSCHEMATC
