File: brd/master/master.sch (KiCad schematic (older format))
At the start: 0 parts

Commit message: master rc3 w/ freecanvas alpha
Parts:
- added C? (x16): 100nF, symbol C
- added C? (x2): 22pF, symbol C
- added C?: 1nF, symbol C
- added C? (x2): 10uF, symbol CP
- added D?: 1N4148, symbol D
- added DS?: LCD16X2, WC1602A, symbol LCD16X2
- added J?: PORTA, symbol CONN_01X08
- added J?: PORTA POWER, symbol CONN_02X08
- added J? (x2): DB9, symbol DB9
- added J?: PORTC, symbol CONN_01X08
- added J?: PORTF, symbol CONN_01X08
- added J?: PORTK, symbol CONN_01X08
- added J?: PORTL, symbol CONN_01X08
- added J?: PORTC POWER, symbol CONN_02X08
- added J?: PORTF POWER, symbol CONN_02X08
- added J?: PORTK POWER, symbol CONN_02X08
- added J?: PORTL POWER, symbol CONN_02X08
- added J?: POWER INPUT, symbol CONN_01X03
- added J?: VCOM, symbol CONN_01X02
- added J?: PORTH, symbol CONN_01X08
- added J?: PORTH POWER, symbol CONN_02X08
- added J?: PORTJ, symbol CONN_01X08
- added J?: PORTJ POWER, symbol CONN_02X08
- added J?: COMM PLUGIN, symbol CONN_02X14
- added P?: ISP, symbol CONN_02X03
- added Q? (x4): BC547, TO-92, symbol BC547
- added Q?: BSS84, symbol Q_PMOS_GSD
- added R?: 1M, symbol R
- added R? (x6): 10k, symbol R
- added R?: 120R, symbol R
- added R?: 100k, symbol R
- added R? (x4): 4k7, symbol R
- added R? (x14): 1k, symbol R
- added RV?: 10k, symbol POT
- added SW?: RESET, symbol SW_PUSH
- added U?: ATMEGA2560-A, TQFP100, symbol ATMEGA2560-A-RESCUE-master
- added U?: MAX13450E, TSSOP-14EP, symbol MAX13450E
- added Y?: 16MHz, symbol Crystal
Connections:
- new net: C?.1, C?.2, D?.2 (A), P?.5 (P5), R?.2, SW?.1, U?.30 (~RESET)
- new net: C?.1, R?.1, U?.33 (XTAL2), Y?.1
- new net: C?.1, R?.2, U?.34 (XTAL1), Y?.2
- new net: C?.1, U?.98 (AREF)
- new net: J?.3, R?.1, U?.10 (Y)
- new net: J?.7 (P7), R?.2, U?.12 (~Z)
- new net: J?.3, U?.8 (A)
- new net: J?.7 (P7), U?.9 (~B)
- new net: J?.1, R?.2
- new net: J?.2, R?.2
- new net: J?.6 (P6), Q?.1 (C)
- new net: J?.8 (P8), J?.8 (P8), Q?.1 (C), R?.2
- new net: J?.2, Q?.1 (C)
- new net: J?.6 (P6), R?.2
- new net: J?.9 (P9), R?.2
- new net: Q?.2 (B), R?.1 (x4)
- new net: Q?.1 (G), R?.1, R?.2
- new net: Q?.2 (S), R?.1
- new net: DS?.16 (LED-), Q?.1 (C)
- new net: DS?.3 (VO), RV?.2
- new net: J?.11 (P11), R?.1
- new net: J?.12 (P12), R?.2
- new net: J?.14 (P14), R?.2
- new net: J?.15 (P15), R?.1
- new net: J?.16 (P16), R?.2
- new net: J?.17 (P17), R?.1
- new net: J?.18 (P18), R?.2
- new net: J?.19 (P19), R?.1
- new net: J?.21 (P21), R?.1
- new net: J?.23 (P23), R?.1
- new net: J?.26 (P26), R?.2
- new net: J?.7 (P7), R?.1
- new net: J?.8 (P8), R?.2
- new net AUX1: R?.1, U?.9 ((CLKO/ICP3/INT7)PE7)
- new net AUX2: R?.1, U?.28 (PG3(TOSC2))
- new net AUX3: R?.1, U?.29 (PG4(TOSC1))
- new net AUX4: R?.2, U?.1 (PG5(OCOB))
- new net CAX1: R?.2, U?.44 ((SDA/INT1)PD1)
- new net CAX2: J?.22 (P22), U?.48 ((XCK1)PD5)
- new net CBX1: R?.2, U?.6 ((OC3B/INT4)PE4)
- new net CBX2: J?.24 (P24), U?.49 ((T1)PD6)
- new net CIDTC: R?.1, U?.7 ((OC3C/INT5)PE5)
- new net CODTC: R?.2, U?.8 ((T3/INT6)PE6)
- new net GND: C?.2, C?.2, C?.2, C?.2, C?.2, C?.2, C?.2, C?.2, C?.2, C?.2, C?.2, C?.2, C?.2, C?.2, C?.2, C?.2, C?.2, C?.2, C?.2, C?.2, DS?.1 (VSS), J?.1, J?.1 (P1), J?.1 (P1), J?.1 (P1), J?.1 (P1), J?.1 (P1), J?.1 (P1), J?.1 (P1), J?.11 (P11), J?.11 (P11), J?.11 (P11), J?.11 (P11), J?.11 (P11), J?.11 (P11), J?.11 (P11), J?.13 (P13), J?.13 (P13), J?.13 (P13), J?.13 (P13), J?.13 (P13), J?.13 (P13), J?.13 (P13), J?.15 (P15), J?.15 (P15), J?.15 (P15), J?.15 (P15), J?.15 (P15), J?.15 (P15), J?.15 (P15), J?.2 (P2), J?.2 (P2), J?.27 (P27), J?.28 (P28), J?.3 (P3), J?.3 (P3), J?.3 (P3), J?.3 (P3), J?.3 (P3), J?.3 (P3), J?.3 (P3), J?.5, J?.5, J?.5 (P5), J?.5 (P5), J?.5 (P5), J?.5 (P5), J?.5 (P5), J?.5 (P5), J?.5 (P5), J?.6 (P6), J?.7 (P7), J?.7 (P7), J?.7 (P7), J?.7 (P7), J?.7 (P7), J?.7 (P7), J?.7 (P7), J?.9 (P9), J?.9 (P9), J?.9 (P9), J?.9 (P9), J?.9 (P9), J?.9 (P9), J?.9 (P9), J?.9 (P9), P?.6 (P6), Q?.3 (E), Q?.3 (E), Q?.3 (E), Q?.3 (E), RV?.3, SW?.2, U?.11 (GND), U?.11 (GND), U?.13 (TERM100), U?.2 (~RE), U?.32 (GND), U?.5 (~TERM), U?.62 (GND), U?.81 (GND), U?.99 (AGND)
- new net INT: R?.2, U?.43 ((SCL/INT0)PD0)
- new net IRQ: J?.20 (P20), U?.47 ((ICP1)PD4)
- new net MDTC: J?.13 (P13), U?.4 ((XCK0/AIN0)PE2)
- new net MISO: J?.1 (P1), P?.1 (P1), U?.22 ((PCINT3/MISO)PB3)
- new net MIU: J?.25 (P25), U?.50 ((T2)PD7)
- new net MOSI: J?.4 (P4), P?.4 (P4), U?.21 ((PCINT2/MOSI)PB2)
- new net PA0: J?.1 (P1), U?.78 ((AD0)PA0)
- new net PA1: J?.2 (P2), U?.77 ((AD1)PA1)
- new net PA2: J?.3 (P3), U?.76 ((AD2)PA2)
- new net PA3: J?.4 (P4), U?.75 ((AD3)PA3)
- new net PA4: J?.5 (P5), U?.74 ((AD4)PA4)
- new net PA5: J?.6 (P6), U?.73 ((AD5)PA5)
- new net PA6: J?.7 (P7), U?.72 ((AD6)PA6)
- new net PA7: J?.8 (P8), U?.71 ((AD7)PA7)
- new net PB4: DS?.11 (D4), U?.23 ((PCINT4/OC2A)PB4)
- new net PB5: DS?.12 (D5), U?.24 ((PCINT5/OC1A)PB5)
- new net PB6: DS?.13 (D6), U?.25 ((PCINT6/OC1B)PB6)
- new net PB7: DS?.14 (D7), U?.26 ((PCINT7/OC0A/OC1C)PB7)
- new net PC0: J?.1 (P1), U?.53 ((A8)PC0)
- new net PC1: J?.2 (P2), U?.54 ((A9)PC1)
- new net PC2: J?.3 (P3), U?.55 ((A10)PC2)
- new net PC3: J?.4 (P4), U?.56 ((A11)PC3)
- new net PC4: J?.5 (P5), U?.57 ((A12)PC4)
- new net PC5: J?.6 (P6), U?.58 ((A13)PC5)
- new net PC6: J?.7 (P7), U?.59 ((A14)PC6)
- new net PC7: J?.8 (P8), U?.60 ((A15)PC7)
- new net PE3: R?.2, U?.5 ((OC3A/AIN1)PE3)
- new net PF0: J?.1 (P1), U?.97 ((ADC0)PF0)
- new net PF1: J?.2 (P2), U?.96 ((ADC1)PF1)
- new net PF2: J?.3 (P3), U?.95 ((ADC2)PF2)
- new net PF3: J?.4 (P4), U?.94 ((ADC3)PF3)
- new net PF4: J?.5 (P5), U?.93 ((TCK/ADC4)PF4)
- new net PF5: J?.6 (P6), U?.92 ((TMS/ADC5)PF5)
- new net PF6: J?.7 (P7), U?.91 ((TD0/ADC6)PF6)
- new net PF7: J?.8 (P8), U?.90 ((TDI/ADC7)PF7)
- new net PG0: DS?.4 (RS), U?.51 (PG0(~WR~))
- new net PG1: DS?.5 (R/W), U?.52 (PG1(~RD~))
- new net PG2: DS?.6 (E), U?.70 (PG2(ALE))
- new net PH0: J?.1 (P1), U?.12 (PH0(RXD2))
- new net PH1: J?.2 (P2), U?.13 (PH1(TXD2))
- new net PH2: J?.3 (P3), U?.14 (PH2(XCK2))
- new net PH3: J?.4 (P4), U?.15 (PH3(OC4A))
- new net PH4: J?.5 (P5), U?.16 (PH4(OC4B))
- new net PH5: J?.6 (P6), U?.17 (PH5(OC4C))
- new net PH6: J?.7 (P7), U?.18 (PH6(OC2B))
- new net PH7: J?.8 (P8), U?.27 (PH7(T4))
- new net PJ0: J?.1 (P1), U?.63 (PJ0(RXD3/PCINT9))
- new net PJ1: J?.2 (P2), U?.64 (PJ1(TXD3/PCINT10))
- new net PJ2: J?.3 (P3), U?.65 (PJ2(XCK3/PCINT11))
- new net PJ3: J?.4 (P4), U?.66 (PJ3(PCINT12))
- new net PJ4: J?.5 (P5), U?.67 (PJ4(PCINT13))
- new net PJ5: J?.6 (P6), U?.68 (PJ5(PCINT14))
- new net PJ6: J?.7 (P7), U?.69 (PJ6(PCINT15))
- new net PJ7: J?.8 (P8), U?.79 (PJ7)
- new net PK0: J?.1 (P1), U?.89 (PK0(ADC8/PCINT16))
- new net PK1: J?.2 (P2), U?.88 (PK1(ADC9/PCINT17))
- new net PK2: J?.3 (P3), U?.87 (PK2(ADC10/PCINT18))
- new net PK3: J?.4 (P4), U?.86 (PK3(ADC11/PCINT19))
- new net PK4: J?.5 (P5), U?.85 (PK4(ADC12/PCINT20))
- new net PK5: J?.6 (P6), U?.84 (PK5(ADC13/PCINT21))
- new net PK6: J?.7 (P7), U?.83 (PK6(ADC14/PCINT22))
- new net PK7: J?.8 (P8), U?.82 (PK7(ADC15/PCINT23))
- new net PL0: J?.1 (P1), U?.35 (PL0(ICP4))
- new net PL1: J?.2 (P2), U?.36 (PL1(ICP5))
- new net PL2: J?.3 (P3), U?.37 (PL2(T5))
- new net PL3: J?.4 (P4), U?.38 (PL3(OC5A))
- new net PL4: J?.5 (P5), U?.39 (PL4(OC5B))
- new net PL5: J?.6 (P6), U?.40 (PL5(OC5C))
- new net PL6: J?.7 (P7), U?.41 (PL6)
- new net PL7: J?.8 (P8), U?.42 (PL7)
- new net PSON: J?.3 (P3), U?.19 ((PCINT0/~SS~)PB0)
- new net REXT: C?.1, J?.5 (P5)
- new net RXD0: R?.2, U?.2 ((PCINT8/RXD0)PE0)
- new net RXD1: R?.1, U?.45 ((RXD1/INT2)PD2)
- new net SCK: J?.3 (P3), P?.3 (P3), U?.20 ((PCINT1/SCK)PB1)
- new net TXD0: R?.1, U?.3 ((TXD0)PE1)
- new net TXD1: R?.2, U?.46 ((TXD1/INT3)PD3)
- new net VCC: C?.1, C?.1, C?.1, C?.1, C?.1, C?.1, C?.1, D?.1 (K), DS?.15 (LED+), DS?.2 (VDD), J?.1 (P1), J?.10 (P10), J?.2 (P2), J?.9 (P9), P?.2 (P2), Q?.3 (D), R?.1, R?.1, R?.1, R?.1, R?.1, R?.1, RV?.1, U?.1 (DE), U?.10 (VCC), U?.100 (AVCC), U?.14 (SRL), U?.31 (VCC), U?.4 (VCC), U?.6 (VL), U?.61 (VCC), U?.80 (VCC)
- new net VCOM: C?.1, C?.1, C?.1, C?.1, C?.1, C?.1, C?.1, C?.1, C?.1, J?.1 (P1), J?.10 (P10), J?.10 (P10), J?.10 (P10), J?.10 (P10), J?.10 (P10), J?.10 (P10), J?.10 (P10), J?.12 (P12), J?.12 (P12), J?.12 (P12), J?.12 (P12), J?.12 (P12), J?.12 (P12), J?.12 (P12), J?.14 (P14), J?.14 (P14), J?.14 (P14), J?.14 (P14), J?.14 (P14), J?.14 (P14), J?.14 (P14), J?.16 (P16), J?.16 (P16), J?.16 (P16), J?.16 (P16), J?.16 (P16), J?.16 (P16), J?.16 (P16), J?.2 (P2), J?.2 (P2), J?.2 (P2), J?.2 (P2), J?.2 (P2), J?.2 (P2), J?.2 (P2), J?.4 (P4), J?.4 (P4), J?.4 (P4), J?.4 (P4), J?.4 (P4), J?.4 (P4), J?.4 (P4), J?.6 (P6), J?.6 (P6), J?.6 (P6), J?.6 (P6), J?.6 (P6), J?.6 (P6), J?.6 (P6), J?.8 (P8), J?.8 (P8), J?.8 (P8), J?.8 (P8), J?.8 (P8), J?.8 (P8), J?.8 (P8)
